Commit message: 2026/09/04

File: install/independent_steering/share/independent_steering/urdf/tr.urdf (robot description, URDF)
Before this commit: robot tr_robot, 9 links, 8 joints
Joints:
- joint lb_wheel_joint: origin xyz=0 0 -0.08 -> xyz=0 0 -0.10
- joint lf_wheel_joint: origin xyz=0 0 -0.08 -> xyz=0 0 -0.10
- joint rb_wheel_joint: origin xyz=0 0 -0.08 -> xyz=0 0 -0.10
- joint rf_wheel_joint: origin xyz=0 0 -0.08 -> xyz=0 0 -0.10
